File: ECE_362_mini_project1.brd (EAGLE design)
At the start: 59.7 x 56.8 mm, 18 parts

Commit message: Updated the board
Parts:
- added R3, R4: (no value), resistor:R0603
- moved JP5 81.0 mm to (54.6, 30.5), turned to 180 degrees
- moved JP4 71.6 mm to (68.6, 11.4), turned to 270 degrees
- moved JP3 66.7 mm to (54.6, 25.4), turned to 180 degrees
- moved C1 64.9 mm to (58.4, 17.8), turned to 180 degrees
- moved U$6 64.4 mm to (61.0, 15.2), turned to 180 degrees
- moved C2 62.7 mm to (53.3, 17.8), turned to 180 degrees
- moved U$3 61.5 mm to (54.6, 5.08), turned to 90 degrees
- moved U$5 34.5 mm to (17.8, 27.9), turned to 180 degrees
- moved U$1 29.7 mm to (3.81, 3.81), turned to 0 degrees
- moved U$2 28.4 mm to (17.8, 27.9), flipped to the bottom, turned to 180 degrees
- moved U$4 17.3 mm to (31.8, 27.9), turned to 180 degrees
- moved JP2 11.5 mm to (22.9, 14.0), turned to 0 degrees
- moved BOOT_SW 4.02 mm to (6.35, 25.4), turned to 180 degrees
- moved R1 2.54 mm to (7.62, 29.2)
- moved R2 2.54 mm to (7.62, 31.8)
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Connections:
- removed net N$5: U$4.9, U$5.15
- net +5V: now also R3.2, R4.2
- net LCD_Q0: now also U$4.9, U$5.15
- net LCD_Q1: now also U$5.1
- net LCD_Q2: now also U$5.2
- net LCD_Q3: now also U$5.3
- net LCD_Q4: now also U$5.4
- net LCD_Q5: now also U$5.5
- net LCD_Q6: now also U$5.6
- net LCD_Q7: now also U$5.7
- net PE0: now also R3.1
- net PE1: now also R4.1
Routing:
- net VIN: track 0.00 -> 5.08 mm
- net TX: track 0.00 -> 5.08 mm
- net RX: track 0.00 -> 5.08 mm
- net RESET: track 0.00 -> 5.08 mm
- net PT7: track 0.00 -> 5.08 mm
- net PT6: track 0.00 -> 5.08 mm
- net PT5: track 0.00 -> 5.08 mm
- net PT4: track 0.00 -> 5.08 mm
- net PT3: track 0.00 -> 5.08 mm
- net PT2: track 0.00 -> 5.08 mm
- net PT1: track 0.00 -> 5.08 mm
- net PT0: track 0.00 -> 5.08 mm
- net PM5: track 0.00 -> 5.08 mm
- net PM4: track 0.00 -> 5.08 mm
- net PM3: track 0.00 -> 5.08 mm
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Other:
- board size 59.7 x 56.8 mm -> 71.1 x 35.2 mm
