File: ECE_362_mini_project2.brd (EAGLE design)
At the start: 70.8 x 34.5 mm, 30 parts

Commit message: cosmetic changes
Parts:
- flipped R12 to the bottom
Routing:
- net LED1_Q7: track 4.66 -> 2.96 mm
- net A7: track 7.92 -> 6.22 mm, vias 1 -> 0
Other:
- board size 70.8 x 34.5 mm -> 70.3 x 34.5 mm
Changed lines of the file:
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@@
 <board>
 <plain>
-<wire x1="0" y1="0" x2="70.084" y2="0.254" width="0" layer="20"/>
-<wire x1="70.084" y1="0.254" x2="70.592" y2="34.468" width="0" layer="20"/>
-<wire x1="70.592" y1="34.468" x2="-0.254" y2="34.468" width="0" layer="20"/>
-<wire x1="-0.254" y1="34.468" x2="0" y2="0" width="0" layer="20"/>
+<wire x1="0" y1="0" x2="70.338" y2="0" width="0" layer="20"/>
+<wire x1="70.338" y1="0" x2="70.338" y2="34.468" width="0" layer="20"/>
+<wire x1="70.338" y1="34.468" x2="0" y2="34.468" width="0" layer="20"/>
+<wire x1="0" y1="34.468" x2="0" y2="0" width="0" layer="20"/>
 <text x="45.466" y="22.86" size="1.016" layer="112">LCD Q0</text>
 <text x="63.5" y="22.86" size="1.016" layer="112">LCD Q7</text>
@@
 <element name="R10" library="resistor" package="R0603" value="220" x="63.5" y="8.382" smashed="yes" rot="MR180"/>
 <element name="R11" library="resistor" package="R0603" value="220" x="63.5" y="5.842" smashed="yes" rot="MR180"/>
-<element name="R12" library="resistor" package="R0603" value="220" x="63.5" y="3.302" smashed="yes" rot="R180"/>
+<element name="R12" library="resistor" package="R0603" value="220" x="63.5" y="3.302" smashed="yes" rot="MR180"/>
 <element name="R20" library="resistor" package="R0603" value="220" x="63.5" y="21.082" smashed="yes" rot="MR180"/>
 <element name="R13" library="resistor" package="R0603" value="220" x="9.906" y="23.876" smashed="yes"/>
@@
 <contactref element="JP6" pad="1"/>
 <polygon width="0.4064" layer="16">
-<vertex x="-0.762" y="0"/>
+<vertex x="-3.302" y="-1.016"/>
 <vertex x="70.612" y="0"/>
 <vertex x="71.628" y="36.322"/>
@@
 <polygon width="0.4064" layer="1">
 <vertex x="-0.254" y="34.544"/>
-<vertex x="70.612" y="34.29"/>
+<vertex x="71.12" y="35.306"/>
 <vertex x="70.612" y="0"/>
 <vertex x="-0.762" y="0.254"/>
 </polygon>
 <via x="46.228" y="19.812" extent="1-16" drill="0.6"/>
-<via x="58.42" y="19.05" extent="1-16" drill="0.6"/>
-<via x="58.166" y="2.286" extent="1-16" drill="0.6"/>
-<via x="46.482" y="2.794" extent="1-16" drill="0.6"/>
+<via x="60.96" y="21.336" extent="1-16" drill="0.6"/>
+<via x="58.42" y="2.54" extent="1-16" drill="0.6"/>
+<via x="46.482" y="2.54" extent="1-16" drill="0.6"/>
 <via x="67.31" y="28.702" extent="1-16" drill="0.6"/>
-<via x="11.938" y="32.004" extent="1-16" drill="0.6"/>
-<via x="8.128" y="32.258" extent="1-16" drill="0.6"/>
+<via x="12.192" y="32.258" extent="1-16" drill="0.6"/>
+<via x="4.064" y="32.766" extent="1-16" drill="0.6"/>
 <contactref element="C3" pad="2"/>
 </signal>
@@
 <wire x1="44.958" y1="8.382" x2="48.514" y2="8.382" width="0.4064" layer="16"/>
 <wire x1="48.514" y1="8.382" x2="48.641" y2="8.509" width="0.4064" layer="16"/>
-<wire x1="48.641" y1="8.509" x2="54.229" y2="8.509" width="0.4064" layer="16"/>
-<wire x1="54.229" y1="8.509" x2="54.61" y2="8.89" width="0.4064" layer="16"/>
-<via x="54.61" y="8.89" extent="1-16" drill="0.6"/>
-<wire x1="57.531" y1="8.509" x2="54.991" y2="8.509" width="0.4064" layer="1"/>
-<wire x1="54.991" y1="8.509" x2="54.61" y2="8.89" width="0.4064" layer="1"/>
+<wire x1="48.641" y1="8.509" x2="54.483" y2="8.509" width="0.4064" layer="16"/>
+<wire x1="54.483" y1="8.509" x2="55.118" y2="8.636" width="0.4064" layer="16"/>
+<via x="55.118" y="8.636" extent="1-16" drill="0.6"/>
+<wire x1="57.531" y1="8.509" x2="55.753" y2="8.509" width="0.4064" layer="1"/>
+<wire x1="55.753" y1="8.509" x2="55.118" y2="8.636" width="0.4064" layer="1"/>
 <contactref element="C3" pad="1"/>
 <wire x1="45.974" y1="15.152" x2="45.974" y2="14.224" width="0.4064" layer="16"/>
@@
 <wire x1="42.672" y1="1.778" x2="36.322" y2="1.778" width="0.4064" layer="16"/>
 <wire x1="36.322" y1="1.778" x2="34.29" y2="3.81" width="0.4064" layer="16"/>
-<wire x1="48.641" y1="7.239" x2="54.229" y2="7.239" width="0.4064" layer="16"/>
-<wire x1="54.229" y1="7.239" x2="54.61" y2="7.366" width="0.4064" layer="16"/>
+<wire x1="48.641" y1="7.239" x2="54.229" y2="7.493" width="0.4064" layer="16"/>
+<wire x1="54.229" y1="7.493" x2="54.61" y2="7.366" width="0.4064" layer="16"/>
 <via x="54.61" y="7.366" extent="1-16" drill="0.6"/>
 <wire x1="54.61" y1="7.366" x2="57.404" y2="7.366" width="0.4064" layer="1"/>
@@
 <wire x1="36.83" y1="8.89" x2="36.83" y2="10.414" width="0.4064" layer="1"/>
 <wire x1="36.83" y1="10.414" x2="37.338" y2="10.922" width="0.4064" layer="1"/>
-<wire x1="37.338" y1="10.922" x2="44.704" y2="10.922" width="0.4064" layer="1"/>
-<via x="44.704" y="10.922" extent="1-16" drill="0.6"/>
-<wire x1="44.704" y1="10.922" x2="48.514" y2="10.922" width="0.4064" layer="16"/>
+<wire x1="37.338" y1="10.922" x2="45.212" y2="10.922" width="0.4064" layer="1"/>
+<via x="45.212" y="10.922" extent="1-16" drill="0.6"/>
+<wire x1="45.212" y1="10.922" x2="48.514" y2="10.922" width="0.4064" layer="16"/>
 <wire x1="48.514" y1="10.922" x2="48.641" y2="11.049" width="0.4064" layer="16"/>
 </signal>
@@
 <contactref element="BOOT_SW" pad="1"/>
 <wire x1="8.89" y1="19.05" x2="8.89" y2="13.97" width="0.4064" layer="1"/>
-<wire x1="8.89" y1="19.05" x2="8.89" y2="21.082" width="0.4064" layer="1"/>
-<wire x1="8.89" y1="21.082" x2="8.89" y2="21.336" width="0.4064" layer="1"/>
+<wire x1="8.89" y1="19.05" x2="8.89" y2="21.336" width="0.4064" layer="1"/>
 <wire x1="8.89" y1="21.336" x2="6.35" y2="23.876" width="0.4064" layer="1"/>
 <wire x1="6.35" y1="23.876" x2="3.816" y2="23.876" width="0.4064" layer="1"/>
@@
 <wire x1="48.514" y1="14.224" x2="48.514" y2="13.716" width="0.8128" layer="16"/>
 <wire x1="48.514" y1="13.716" x2="48.641" y2="13.589" width="0.4064" layer="16"/>
-<wire x1="57.531" y1="5.969" x2="54.483" y2="5.969" width="0.4064" layer="1"/>
-<wire x1="54.483" y1="5.969" x2="53.594" y2="5.08" width="0.4064" layer="1"/>
-<wire x1="53.594" y1="5.08" x2="52.07" y2="5.08" width="0.8128" layer="1"/>
-<wire x1="52.07" y1="5.08" x2="51.562" y2="5.588" width="0.8128" layer="1"/>
-<via x="51.562" y="5.588" extent="1-16" drill="0.6"/>
-<wire x1="51.562" y1="5.588" x2="51.181" y2="5.969" width="0.8128" layer="16"/>
+<wire x1="57.531" y1="5.969" x2="56.261" y2="5.969" width="0.4064" layer="1"/>
+<wire x1="56.261" y1="5.969" x2="54.61" y2="5.08" width="0.4064" layer="1"/>
+<wire x1="54.61" y1="5.08" x2="52.07" y2="5.08" width="0.8128" layer="1"/>
+<wire x1="52.07" y1="5.08" x2="51.308" y2="5.842" width="0.8128" layer="1"/>
+<via x="51.308" y="5.842" extent="1-16" drill="0.6"/>
+<wire x1="51.308" y1="5.842" x2="51.181" y2="5.969" width="0.8128" layer="16"/>
 <wire x1="51.181" y1="5.969" x2="48.641" y2="5.969" width="0.8128" layer="16"/>
 <wire x1="48.641" y1="5.969" x2="47.117" y2="5.969" width="0.8128" layer="16"/>
-<wire x1="47.117" y1="5.969" x2="46.736" y2="6.35" width="0.8128" layer="16"/>
-<via x="46.736" y="6.35" extent="1-16" drill="0.6"/>
+<wire x1="47.117" y1="5.969" x2="46.736" y2="6.096" width="0.8128" layer="16"/>
+<via x="46.736" y="6.096" extent="1-16" drill="0.6"/>
 <contactref element="R13" pad="2"/>
 <wire x1="10.756" y1="23.876" x2="11.43" y2="23.202" width="0.4064" layer="1"/>
 <wire x1="11.43" y1="23.202" x2="11.43" y2="19.05" width="0.4064" layer="1"/>
-<wire x1="46.736" y1="6.35" x2="46.736" y2="12.954" width="0.8128" layer="1"/>
+<wire x1="46.736" y1="6.096" x2="46.736" y2="12.954" width="0.8128" layer="1"/>
 <via x="46.736" y="12.954" extent="1-16" drill="0.6"/>
 <wire x1="46.736" y1="12.954" x2="47.244" y2="13.462" width="0.8128" layer="16"/>
@@
 <contactref element="JP3" pad="8"/>
 <contactref element="R12" pad="2"/>
-<wire x1="62.65" y1="3.302" x2="67.31" y2="3.302" width="0.4064" layer="1"/>
+<wire x1="64.35" y1="3.302" x2="67.31" y2="3.302" width="0.4064" layer="16"/>
 </signal>
 <signal name="LCD_Q0">
@@
 <wire x1="48.641" y1="4.699" x2="51.943" y2="4.699" width="0.4064" layer="16"/>
 <wire x1="51.943" y1="4.699" x2="53.594" y2="6.35" width="0.4064" layer="16"/>
-<via x="53.594" y="6.35" extent="1-16" drill="0.6"/>
+<via x="53.594" y="6.35" extent="1-16" drill="0.5"/>
 <wire x1="53.594" y1="6.35" x2="53.594" y2="9.144" width="0.4064" layer="1"/>
 <wire x1="53.594" y1="9.144" x2="55.372" y2="10.922" width="0.4064" layer="1"/>
@@
 <contactref element="U$2" pad="7"/>
 <contactref element="R12" pad="1"/>
-<wire x1="64.35" y1="3.302" x2="61.214" y2="3.302" width="0.4064" layer="1"/>
-<wire x1="61.214" y1="3.302" x2="58.674" y2="5.842" width="0.4064" layer="16"/>
-<wire x1="58.674" y1="5.842" x2="57.658" y2="5.842" width="0.4064" layer="16"/>
-<wire x1="57.658" y1="5.842" x2="57.531" y2="5.969" width="0.4064" layer="16"/>
-<via x="61.214" y="3.302" extent="1-16" drill="0.6"/>
+<wire x1="57.531" y1="5.969" x2="58.547" y2="5.969" width="0.4064" layer="16"/>
+<wire x1="58.547" y1="5.969" x2="61.214" y2="3.302" width="0.4064" layer="16"/>
+<wire x1="61.214" y1="3.302" x2="62.65" y2="3.302" width="0.4064" layer="16"/>
 </signal>
 <signal name="A0">
