File: ECE_362_mini_project2.sch (EAGLE design)
At the start: 18 parts

Commit message: Updated the board
Parts:
- removed JP4: (no value), pinhead:PINHD-1X8
- removed U$4: SHIFT_REGISTER, mini_project_parts:SHIFT_REGISTER
- added JP6: (no value), pinhead:PINHD-1X8
- added R10, R11, R12, R20, R5, R6, R7, R8, R9: 220, resistor:R-US_R0603
- added R3, R4: 10k, resistor:R-US_R0603
Connections:
- removed net LED2_Q0: JP4.1
- removed net LED2_Q1: JP4.2
- removed net LED2_Q2: JP4.3
- removed net LED2_Q3: JP4.4
- removed net LED2_Q4: JP4.5
- removed net LED2_Q5: JP4.6
- removed net LED2_Q6: JP4.7
- removed net LED2_Q7: JP4.8
- new net A0: R20.1, U$2.Q0
- new net A1: R6.1, U$2.Q1
- new net A2: R7.1, U$2.Q2
- new net A3: R8.1, U$2.Q3
- new net A4: R9.1, U$2.Q4
- new net A5: R10.1, U$2.Q5
- new net A7: R12.1, U$2.Q7
- new net N$3: R11.1, U$2.Q6
- new net N$9: JP6.7, R5.2
- net +5V: now also JP6.2, R3.2, R4.2, R5.1, U$2.MR, U$5.MR; no longer U$4.VIN
- net AN7: now also U$2.STCP, U$5.STCP
- net GND: now also JP6.1, JP6.3, JP6.8, U$2.OE, U$5.OE; no longer U$4.GND
- net LCD_Q0: now also U$5.Q0
- net LCD_Q1: now also U$5.Q1
- net LCD_Q2: now also U$5.Q2
- net LCD_Q3: now also U$5.Q3
- net LCD_Q4: now also U$5.Q4
- net LCD_Q5: now also U$5.Q5
- net LCD_Q6: now also U$5.Q6
- net LCD_Q7: now also U$5.Q7
- net LED1_Q0: now also R20.2
- net LED1_Q1: now also R6.2
- net LED1_Q2: now also R7.2
- net LED1_Q3: now also R8.2
- net LED1_Q4: now also R9.2
- net LED1_Q5: now also R10.2
- net LED1_Q6: now also R11.2
- net LED1_Q7: now also R12.2
- net N$4: now also U$5.DS; no longer U$4.Q0
- net N$5: now also U$2.DS; no longer U$4.Q7S, U$5.Q0
- net PE0: now also R3.1
- net PE1: now also R4.1
- net PM5: now also U$2.SHCP, U$5.SHCP
- net PT2: now also JP6.4
- net PT3: now also JP6.5
- net PT4: now also JP6.6
Other:
- moved on the sheet: JP5
